File: main.sch (EAGLE design)
At the start: 23 parts, among them IC1 MEGA16-A, IC2 MCP73831, IC3 7805DT

Commit message: Schematics
Parts:
- removed C1, C2: 0.1u, rcl:C-EUC1206
- removed Q1: (no value), crystal:CRYSTALTC26H
- added C8, C9: 0.1u, rcl:C-EUC1206
- added Q2: (no value), crystal:CRYSTALTC26H
- added R10, R11, R12, R8, R9: 10k, rcl:R-EU_R1206
- added R13, R14, R15, R16, R17, R18, R19, R20, R21: (no value), rcl:R-EU_R1206
- added R3, R4, R5, R6, R7: 5k, rcl:R-EU_R1206
Connections:
- removed net 0V: C1.1, C2.1
- removed net N$4: IC1.VCC, IC1.VCC1, IC1.VCC2
- removed net N$6: C7.1, IC2.VBAT, JP2.1
- new net +12V: C3.1, D1.C, IC3.VI, R1.1, R20.2
- new net +3V3: C7.1, IC2.VBAT, JP2.1, U$1.VDD
- new net DS1629_SCL: IC1.PC0(SCL), U$1.SCL
- new net DS1629_SDA: IC1.PC1(SDA), U$1.SDA
- new net MCU_CLOCK: IC1.XTAL1, U$1.OSC
- new net N$13: R3.2, R8.1, T1.B
- new net N$14: R4.2, R9.1, T2.B
- new net N$15: R10.1, R5.2, T3.B
- new net N$16: R11.1, R6.2, T4.B
- new net N$17: R12.1, R7.2, T5.B
- new net N$18: LED1.C, LED1.D3, R15.2
- new net N$19: IC1.(INT1)PD3, R17.1
- new net N$20: IC1.(OC2)PD7, R13.1
- new net N$21: IC1.(ICP)PD6, R14.1
- new net N$22: IC1.(OC1A)PD5, R15.1
- new net N$23: IC1.(TOSC1)PC6, R3.1
- new net N$24: IC1.(TDI)PC5, R4.1
- new net N$25: IC1.(TDO)PC4, R5.1
- new net N$26: IC1.(TMS)PC3, R6.1
- new net N$27: IC1.(TCK)PC2, R7.1
- new net N$28: C8.1, Q2.2, U$1.X1
- new net N$29: C9.1, Q2.1, U$1.X2
- new net N$30: IC1.(OC1B)PD4, R16.1
- new net N$31: LED1.D5, LED1.E, R17.2
- new net N$32: LED1.D6, LED1.F, R18.2
- new net N$33: LED1.D8, LED1.G, R19.2
- new net N$34: LED1.A, LED1.D1, R13.2
- new net N$35: IC1.(INT0)PD2, R18.1
- new net N$36: IC1.(TXD)PD1, R19.1
- net +5V: now also C5.1, IC1.VCC, IC1.VCC1, IC1.VCC2, R10.2, R11.2, R12.2, R8.2, R9.2, T1.E, T2.E, T3.E, T4.E, T5.E
- net GND: now also C5.2, C8.2, C9.2, R21.1, U$1.GND
- net N$1: now also LED1.B, LED1.D2, R14.2; no longer C2.2, IC1.XTAL2, Q1.2
- net N$12: now also LED1.COM9
- net N$2: now also LED1.D, LED1.D4, R16.2; no longer C1.2, IC1.XTAL1, Q1.1
- net N$3: now also IC1.(ADC0)PA0, R20.1, R21.2; no longer C3.1, D1.C, IC3.VI, R1.1
Other:
- moved on the sheet: C3, C4, C5, D1, IC3, JP1, LED1, R1, T1, T2, T3, T4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

Commit message: Schematics
Parts:
- removed C4: 0.1u, rcl:C-EUC1206
- added D2: (no value), diode:ZENER-DIODESOT23
- C5: value (none) -> 0.1u
- C6: value (none) -> 4.7u
- C7: value (none) -> 2u
- C8, C9: value 0.1u -> 12p
- R1: device rcl:R-EU_R1206 -> rcl:R-EU_0204/5
- R13, R14, R15, R16, R17, R18, R19: value (none) -> 100
- R2: value (none) -> 13k
Connections:
- removed net CHARGE_LED: IC2.STAT
- removed net N$5: JP1.1, R1.2
- new net N$4: IC1.(ADC7)PA7, IC2.STAT
- net +12V: no longer D1.C, R1.1
- net +5V: now also IC1.GND@1; no longer C4.1
- net GND: now also D2.A; no longer C4.2, D1.A
- net N$3: now also D2.C
Other:
- moved on the sheet: D1, JP1, R1

Commit message: Schematics
Parts:
- removed D1: (no value), diode:ZENER-DIODESOT23
- removed R1: (no value), rcl:R-EU_0204/5
- added D3: (no value), diode:DIODE-DO15-12
Connections:
- new net N$5: D3.A, JP1.1
- net +12V: now also D3.C
Changed lines of the file:
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@@
 <part name="GND1" library="supply1" deviceset="GND" device=""/>
 <part name="GND2" library="supply1" deviceset="GND" device=""/>
-<part name="D1" library="diode" deviceset="ZENER-DIODE" device="SOT23"/>
 <part name="P+1" library="supply1" deviceset="+5V" device=""/>
 <part name="GND3" library="supply1" deviceset="GND" device=""/>
@@
 <part name="P+6" library="supply1" deviceset="+5V" device=""/>
 <part name="D2" library="diode" deviceset="ZENER-DIODE" device="SOT23"/>
-<part name="R1" library="rcl" deviceset="R-EU_" device="0204/5"/>
+<part name="D3" library="diode" deviceset="DIODE-" device="DO15-12"/>
 </parts>
 <sheets>
@@
 <instance part="GND1" gate="1" x="78.74" y="147.32"/>
 <instance part="GND2" gate="1" x="144.78" y="96.52"/>
-<instance part="D1" gate="G$1" x="43.18" y="162.56" rot="R90"/>
 <instance part="P+1" gate="1" x="104.14" y="185.42"/>
 <instance part="GND3" gate="1" x="152.4" y="195.58"/>
@@
 <instance part="P+6" gate="1" x="134.62" y="157.48"/>
 <instance part="D2" gate="G$1" x="220.98" y="139.7" rot="R90"/>
-<instance part="R1" gate="G$1" x="33.02" y="172.72" rot="R90"/>
+<instance part="D3" gate="G$1" x="43.18" y="180.34"/>
 </instances>
 <busses>
@@
 <pinref part="P+4" gate="1" pin="+12V"/>
 <wire x1="58.42" y1="193.04" x2="58.42" y2="180.34" width="0.1524" layer="91"/>
-<wire x1="50.8" y1="180.34" x2="58.42" y2="180.34" width="0.1524" layer="91"/>
+<wire x1="45.72" y1="180.34" x2="58.42" y2="180.34" width="0.1524" layer="91"/>
+<pinref part="D3" gate="G$1" pin="C"/>
 </segment>
 <segment>
@@
 </segment>
 </net>
+<net name="N$5" class="0">
+<segment>
+<pinref part="JP1" gate="G$1" pin="1"/>
+<wire x1="20.32" y1="180.34" x2="40.64" y2="180.34" width="0.1524" layer="91"/>
+<pinref part="D3" gate="G$1" pin="A"/>
+</segment>
+</net>

Commit message: Schematics
Parts:
- added D1: BZX84CSMD, diode:BZX84CSMD
- added R1: 200, rcl:R-EU_M1206
- added R22: 10k, rcl:R-EU_M1206
- added T6: (no value), transistor:-NPN-SOT23-EBC
- C3: value (none) -> 0.33uF
- D2: value (none) -> BZX84CSMD; device diode:ZENER-DIODESOT23 -> diode:BZX84CSMD
Connections:
- new net N$6: D1.C, R1.1, T6.B
- new net N$7: C3.1, IC3.VI, R22.2, T6.E
- net +12V: now also R1.2, T6.C; no longer C3.1, IC3.VI
- net +5V: now also IC1.AVCC, IC1.RESET
- net GND: now also D1.A, R22.1; no longer IC1.RESET
Other:
- moved on the sheet: D3
Changed lines of the file:
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@@
 <part name="IC2" library="microchip-update-2" deviceset="MCP73831" device=""/>
 <part name="IC3" library="linear" deviceset="78*" device="DT" technology="05"/>
-<part name="C3" library="rcl" deviceset="C-EU" device="C1206"/>
+<part name="C3" library="rcl" deviceset="C-EU" device="C1206" value="0.33uF"/>
 <part name="C5" library="rcl" deviceset="C-EU" device="C1206" value="0.1u"/>
 <part name="GND1" library="supply1" deviceset="GND" device=""/>
@@
 <part name="GND8" library="supply1" deviceset="GND" device=""/>
 <part name="P+6" library="supply1" deviceset="+5V" device=""/>
-<part name="D2" library="diode" deviceset="ZENER-DIODE" device="SOT23"/>
 <part name="D3" library="diode" deviceset="DIODE-" device="DO15-12"/>
+<part name="R1" library="rcl" deviceset="R-EU_" device="M1206" value="200"/>
+<part name="D1" library="diode" deviceset="BZX84CSMD" device=""/>
+<part name="T6" library="transistor" deviceset="*-NPN-" device="SOT23-EBC"/>
+<part name="R22" library="rcl" deviceset="R-EU_" device="M1206" value="10k"/>
+<part name="D2" library="diode" deviceset="BZX84CSMD" device=""/>
 </parts>
 <sheets>
@@
 <instance part="R20" gate="G$1" x="213.36" y="154.94" rot="R90"/>
 <instance part="R21" gate="G$1" x="213.36" y="139.7" rot="R90"/>
-<instance part="P+4" gate="1" x="58.42" y="195.58"/>
+<instance part="P+4" gate="1" x="38.1" y="195.58"/>
 <instance part="P+5" gate="1" x="213.36" y="177.8"/>
 <instance part="GND8" gate="1" x="213.36" y="124.46"/>
 <instance part="P+6" gate="1" x="134.62" y="157.48"/>
+<instance part="D3" gate="G$1" x="33.02" y="180.34"/>
+<instance part="R1" gate="G$1" x="38.1" y="170.18" rot="R90"/>
+<instance part="D1" gate="G$1" x="45.72" y="160.02" rot="R90"/>
+<instance part="T6" gate="G$1" x="45.72" y="177.8" rot="R90"/>
+<instance part="R22" gate="G$1" x="55.88" y="167.64" rot="R90"/>
 <instance part="D2" gate="G$1" x="220.98" y="139.7" rot="R90"/>
-<instance part="D3" gate="G$1" x="43.18" y="180.34"/>
 </instances>
 <busses>
@@
 <net name="GND" class="0">
 <segment>
-<pinref part="IC1" gate="G$1" pin="RESET"/>
-<wire x1="152.4" y1="152.4" x2="144.78" y2="152.4" width="0.1524" layer="91"/>
-<wire x1="144.78" y1="152.4" x2="144.78" y2="114.3" width="0.1524" layer="91"/>
 <pinref part="IC1" gate="G$1" pin="GND1"/>
 <wire x1="144.78" y1="114.3" x2="144.78" y2="111.76" width="0.1524" layer="91"/>
@@
 <junction x="144.78" y="109.22"/>
 <junction x="144.78" y="111.76"/>
-<junction x="144.78" y="114.3"/>
 <pinref part="GND2" gate="1" pin="GND"/>
 <pinref part="C5" gate="G$1" pin="2"/>
@@
 <wire x1="27.94" y1="177.8" x2="27.94" y2="154.94" width="0.1524" layer="91"/>
 <pinref part="IC3" gate="A1" pin="GND"/>
-<wire x1="27.94" y1="154.94" x2="66.04" y2="154.94" width="0.1524" layer="91"/>
+<wire x1="27.94" y1="154.94" x2="45.72" y2="154.94" width="0.1524" layer="91"/>
+<wire x1="45.72" y1="154.94" x2="55.88" y2="154.94" width="0.1524" layer="91"/>
+<wire x1="55.88" y1="154.94" x2="66.04" y2="154.94" width="0.1524" layer="91"/>
 <wire x1="66.04" y1="154.94" x2="78.74" y2="154.94" width="0.1524" layer="91"/>
 <wire x1="78.74" y1="154.94" x2="78.74" y2="172.72" width="0.1524" layer="91"/>
@@
 <junction x="78.74" y="154.94"/>
 <pinref part="JP1" gate="G$1" pin="2"/>
+<pinref part="D1" gate="G$1" pin="A"/>
+<wire x1="45.72" y1="157.48" x2="45.72" y2="154.94" width="0.1524" layer="91"/>
+<junction x="45.72" y="154.94"/>
+<pinref part="R22" gate="G$1" pin="1"/>
+<wire x1="55.88" y1="162.56" x2="55.88" y2="154.94" width="0.1524" layer="91"/>
+<junction x="55.88" y="154.94"/>
 </segment>
 <segment>
@@
 <pinref part="R21" gate="G$1" pin="1"/>
 <wire x1="213.36" y1="127" x2="213.36" y2="132.08" width="0.1524" layer="91"/>
-<pinref part="D2" gate="G$1" pin="A"/>
 <wire x1="213.36" y1="132.08" x2="213.36" y2="134.62" width="0.1524" layer="91"/>
 <wire x1="220.98" y1="137.16" x2="220.98" y2="132.08" width="0.1524" layer="91"/>
 <wire x1="220.98" y1="132.08" x2="213.36" y2="132.08" width="0.1524" layer="91"/>
 <junction x="213.36" y="132.08"/>
+<pinref part="D2" gate="G$1" pin="A"/>
 </segment>
 </net>
@@
 <junction x="149.86" y="124.46"/>
 <pinref part="C5" gate="G$1" pin="1"/>
-<wire x1="134.62" y1="129.54" x2="134.62" y2="154.94" width="0.1524" layer="91"/>
+<wire x1="134.62" y1="129.54" x2="134.62" y2="152.4" width="0.1524" layer="91"/>
+<wire x1="134.62" y1="152.4" x2="134.62" y2="154.94" width="0.1524" layer="91"/>
 <wire x1="134.62" y1="124.46" x2="134.62" y2="119.38" width="0.1524" layer="91"/>
 <junction x="134.62" y="124.46"/>
 <pinref part="IC1" gate="G$1" pin="GND@1"/>
-<wire x1="152.4" y1="129.54" x2="134.62" y2="129.54" width="0.1524" layer="91"/>
+<wire x1="152.4" y1="129.54" x2="149.86" y2="129.54" width="0.1524" layer="91"/>
 <junction x="134.62" y="129.54"/>
+<pinref part="IC1" gate="G$1" pin="AVCC"/>
+<wire x1="149.86" y1="129.54" x2="134.62" y2="129.54" width="0.1524" layer="91"/>
+<wire x1="152.4" y1="132.08" x2="149.86" y2="132.08" width="0.1524" layer="91"/>
+<wire x1="149.86" y1="132.08" x2="149.86" y2="129.54" width="0.1524" layer="91"/>
+<junction x="149.86" y="129.54"/>
+<pinref part="IC1" gate="G$1" pin="RESET"/>
+<wire x1="152.4" y1="152.4" x2="134.62" y2="152.4" width="0.1524" layer="91"/>
+<junction x="134.62" y="152.4"/>
 </segment>
 </net>
@@
 <net name="+12V" class="0">
 <segment>
-<pinref part="IC3" gate="A1" pin="VI"/>
-<pinref part="C3" gate="G$1" pin="1"/>
-<wire x1="66.04" y1="180.34" x2="68.58" y2="180.34" width="0.1524" layer="91"/>
-<wire x1="66.04" y1="172.72" x2="66.04" y2="180.34" width="0.1524" layer="91"/>
-<wire x1="58.42" y1="180.34" x2="66.04" y2="180.34" width="0.1524" layer="91"/>
-<junction x="58.42" y="180.34"/>
-<junction x="66.04" y="180.34"/>
-<pinref part="P+4" gate="1" pin="+12V"/>
-<wire x1="58.42" y1="193.04" x2="58.42" y2="180.34" width="0.1524" layer="91"/>
-<wire x1="45.72" y1="180.34" x2="58.42" y2="180.34" width="0.1524" layer="91"/>
-<pinref part="D3" gate="G$1" pin="C"/>
-</segment>
-<segment>
 <pinref part="P+5" gate="1" pin="+12V"/>
 <pinref part="R20" gate="G$1" pin="2"/>
 <wire x1="213.36" y1="175.26" x2="213.36" y2="160.02" width="0.1524" layer="91"/>
+</segment>
+<segment>
+<pinref part="D3" gate="G$1" pin="C"/>
+<wire x1="35.56" y1="180.34" x2="38.1" y2="180.34" width="0.1524" layer="91"/>
+<pinref part="T6" gate="G$1" pin="C"/>
+<pinref part="R1" gate="G$1" pin="2"/>
+<wire x1="38.1" y1="180.34" x2="40.64" y2="180.34" width="0.1524" layer="91"/>
+<wire x1="38.1" y1="175.26" x2="38.1" y2="180.34" width="0.1524" layer="91"/>
+<junction x="38.1" y="180.34"/>
+<pinref part="P+4" gate="1" pin="+12V"/>
+<wire x1="38.1" y1="193.04" x2="38.1" y2="180.34" width="0.1524" layer="91"/>
 </segment>
 </net>
@@
 <wire x1="203.2" y1="147.32" x2="213.36" y2="147.32" width="0.1524" layer="91"/>
 <junction x="213.36" y="147.32"/>
-<pinref part="D2" gate="G$1" pin="C"/>
 <wire x1="213.36" y1="147.32" x2="220.98" y2="147.32" width="0.1524" layer="91"/>
 <wire x1="220.98" y1="147.32" x2="220.98" y2="142.24" width="0.1524" layer="91"/>
+<pinref part="D2" gate="G$1" pin="C"/>
 </segment>
 </net>
@@
 <segment>
 <pinref part="JP1" gate="G$1" pin="1"/>
-<wire x1="20.32" y1="180.34" x2="40.64" y2="180.34" width="0.1524" layer="91"/>
+<wire x1="20.32" y1="180.34" x2="30.48" y2="180.34" width="0.1524" layer="91"/>
 <pinref part="D3" gate="G$1" pin="A"/>
 </segment>
 </net>
+<net name="N$6" class="0">
+<segment>
+<pinref part="R1" gate="G$1" pin="1"/>
+<pinref part="D1" gate="G$1" pin="C"/>
+<wire x1="38.1" y1="165.1" x2="45.72" y2="165.1" width="0.1524" layer="91"/>
+<wire x1="45.72" y1="165.1" x2="45.72" y2="162.56" width="0.1524" layer="91"/>
+<pinref part="T6" gate="G$1" pin="B"/>
+<wire x1="45.72" y1="175.26" x2="45.72" y2="165.1" width="0.1524" layer="91"/>
+<junction x="45.72" y="165.1"/>
+</segment>
+</net>
+<net name="N$7" class="0">
+<segment>
+<pinref part="IC3" gate="A1" pin="VI"/>
+<pinref part="C3" gate="G$1" pin="1"/>
+<wire x1="66.04" y1="180.34" x2="68.58" y2="180.34" width="0.1524" layer="91"/>
+<wire x1="66.04" y1="172.72" x2="66.04" y2="180.34" width="0.1524" layer="91"/>
+<wire x1="55.88" y1="180.34" x2="66.04" y2="180.34" width="0.1524" layer="91"/>
+<junction x="66.04" y="180.34"/>
+<junction x="55.88" y="180.34"/>
+<wire x1="50.8" y1="180.34" x2="55.88" y2="180.34" width="0.1524" layer="91"/>
+<pinref part="T6" gate="G$1" pin="E"/>
+<pinref part="R22" gate="G$1" pin="2"/>
+<wire x1="55.88" y1="172.72" x2="55.88" y2="180.34" width="0.1524" layer="91"/>
+</segment>
+</net>

Commit message: Schematics
Parts:
- removed R22: 10k, rcl:R-EU_M1206
- R20: value (none) -> 1.3k
- R21: value (none) -> 500
Connections:
- net +5V: now also IC1.AREF
- net GND: no longer R22.1
- net N$7: no longer R22.2
Changed lines of the file:
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@@
 <part name="R19" library="rcl" deviceset="R-EU_" device="R1206" value="100"/>
 <part name="+3V2" library="supply1" deviceset="+3V3" device=""/>
-<part name="R20" library="rcl" deviceset="R-EU_" device="R1206"/>
-<part name="R21" library="rcl" deviceset="R-EU_" device="R1206"/>
+<part name="R20" library="rcl" deviceset="R-EU_" device="R1206" value="1.3k"/>
+<part name="R21" library="rcl" deviceset="R-EU_" device="R1206" value="500"/>
 <part name="P+4" library="supply1" deviceset="+12V" device=""/>
 <part name="P+5" library="supply1" deviceset="+12V" device=""/>
@@
 <part name="D1" library="diode" deviceset="BZX84CSMD" device=""/>
 <part name="T6" library="transistor" deviceset="*-NPN-" device="SOT23-EBC"/>
-<part name="R22" library="rcl" deviceset="R-EU_" device="M1206" value="10k"/>
 <part name="D2" library="diode" deviceset="BZX84CSMD" device=""/>
 </parts>
@@
 <instance part="D1" gate="G$1" x="45.72" y="160.02" rot="R90"/>
 <instance part="T6" gate="G$1" x="45.72" y="177.8" rot="R90"/>
-<instance part="R22" gate="G$1" x="55.88" y="167.64" rot="R90"/>
 <instance part="D2" gate="G$1" x="220.98" y="139.7" rot="R90"/>
 </instances>
@@
 <pinref part="IC3" gate="A1" pin="GND"/>
 <wire x1="27.94" y1="154.94" x2="45.72" y2="154.94" width="0.1524" layer="91"/>
-<wire x1="45.72" y1="154.94" x2="55.88" y2="154.94" width="0.1524" layer="91"/>
-<wire x1="55.88" y1="154.94" x2="66.04" y2="154.94" width="0.1524" layer="91"/>
+<wire x1="45.72" y1="154.94" x2="66.04" y2="154.94" width="0.1524" layer="91"/>
 <wire x1="66.04" y1="154.94" x2="78.74" y2="154.94" width="0.1524" layer="91"/>
 <wire x1="78.74" y1="154.94" x2="78.74" y2="172.72" width="0.1524" layer="91"/>
@@
 <wire x1="45.72" y1="157.48" x2="45.72" y2="154.94" width="0.1524" layer="91"/>
 <junction x="45.72" y="154.94"/>
-<pinref part="R22" gate="G$1" pin="1"/>
-<wire x1="55.88" y1="162.56" x2="55.88" y2="154.94" width="0.1524" layer="91"/>
-<junction x="55.88" y="154.94"/>
 </segment>
 <segment>
@@
 <junction x="149.86" y="124.46"/>
 <pinref part="C5" gate="G$1" pin="1"/>
-<wire x1="134.62" y1="129.54" x2="134.62" y2="152.4" width="0.1524" layer="91"/>
+<wire x1="134.62" y1="129.54" x2="134.62" y2="134.62" width="0.1524" layer="91"/>
+<wire x1="134.62" y1="134.62" x2="134.62" y2="152.4" width="0.1524" layer="91"/>
 <wire x1="134.62" y1="152.4" x2="134.62" y2="154.94" width="0.1524" layer="91"/>
 <wire x1="134.62" y1="124.46" x2="134.62" y2="119.38" width="0.1524" layer="91"/>
@@
 <wire x1="152.4" y1="152.4" x2="134.62" y2="152.4" width="0.1524" layer="91"/>
 <junction x="134.62" y="152.4"/>
+<pinref part="IC1" gate="G$1" pin="AREF"/>
+<wire x1="152.4" y1="134.62" x2="134.62" y2="134.62" width="0.1524" layer="91"/>
+<junction x="134.62" y="134.62"/>
 </segment>
 </net>
@@
 <wire x1="66.04" y1="180.34" x2="68.58" y2="180.34" width="0.1524" layer="91"/>
 <wire x1="66.04" y1="172.72" x2="66.04" y2="180.34" width="0.1524" layer="91"/>
-<wire x1="55.88" y1="180.34" x2="66.04" y2="180.34" width="0.1524" layer="91"/>
+<wire x1="50.8" y1="180.34" x2="66.04" y2="180.34" width="0.1524" layer="91"/>
 <junction x="66.04" y="180.34"/>
-<junction x="55.88" y="180.34"/>
-<wire x1="50.8" y1="180.34" x2="55.88" y2="180.34" width="0.1524" layer="91"/>
 <pinref part="T6" gate="G$1" pin="E"/>
-<pinref part="R22" gate="G$1" pin="2"/>
-<wire x1="55.88" y1="172.72" x2="55.88" y2="180.34" width="0.1524" layer="91"/>
-</segment>
-</net>
+</segment>
+</net>

Commit message: Schematics
Parts:
- Q2: value (none) -> 32768k
Connections:
- net +5V: no longer IC1.GND@1
- net GND: now also IC1.GND@1
Changed lines of the file:
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@@
 <part name="R11" library="rcl" deviceset="R-EU_" device="R1206" value="10k"/>
 <part name="R12" library="rcl" deviceset="R-EU_" device="R1206" value="10k"/>
-<part name="Q2" library="crystal" deviceset="CRYSTAL" device="TC26H"/>
+<part name="Q2" library="crystal" deviceset="CRYSTAL" device="TC26H" value="32768k"/>
 <part name="C8" library="rcl" deviceset="C-EU" device="C1206" value="12p"/>
 <part name="C9" library="rcl" deviceset="C-EU" device="C1206" value="12p"/>
@@
 <wire x1="134.62" y1="111.76" x2="134.62" y2="109.22" width="0.1524" layer="91"/>
 <wire x1="134.62" y1="109.22" x2="144.78" y2="109.22" width="0.1524" layer="91"/>
+<pinref part="IC1" gate="G$1" pin="GND@1"/>
+<wire x1="152.4" y1="129.54" x2="144.78" y2="129.54" width="0.1524" layer="91"/>
+<wire x1="144.78" y1="129.54" x2="144.78" y2="114.3" width="0.1524" layer="91"/>
+<junction x="144.78" y="114.3"/>
 </segment>
 <segment>
@@
 <pinref part="P+6" gate="1" pin="+5V"/>
 <wire x1="149.86" y1="124.46" x2="134.62" y2="124.46" width="0.1524" layer="91"/>
-<wire x1="134.62" y1="124.46" x2="134.62" y2="129.54" width="0.1524" layer="91"/>
 <junction x="149.86" y="124.46"/>
 <pinref part="C5" gate="G$1" pin="1"/>
-<wire x1="134.62" y1="129.54" x2="134.62" y2="134.62" width="0.1524" layer="91"/>
+<wire x1="134.62" y1="124.46" x2="134.62" y2="132.08" width="0.1524" layer="91"/>
+<wire x1="134.62" y1="132.08" x2="134.62" y2="134.62" width="0.1524" layer="91"/>
 <wire x1="134.62" y1="134.62" x2="134.62" y2="152.4" width="0.1524" layer="91"/>
 <wire x1="134.62" y1="152.4" x2="134.62" y2="154.94" width="0.1524" layer="91"/>
 <wire x1="134.62" y1="124.46" x2="134.62" y2="119.38" width="0.1524" layer="91"/>
 <junction x="134.62" y="124.46"/>
-<pinref part="IC1" gate="G$1" pin="GND@1"/>
-<wire x1="152.4" y1="129.54" x2="149.86" y2="129.54" width="0.1524" layer="91"/>
-<junction x="134.62" y="129.54"/>
-<pinref part="IC1" gate="G$1" pin="AVCC"/>
-<wire x1="149.86" y1="129.54" x2="134.62" y2="129.54" width="0.1524" layer="91"/>
-<wire x1="152.4" y1="132.08" x2="149.86" y2="132.08" width="0.1524" layer="91"/>
-<wire x1="149.86" y1="132.08" x2="149.86" y2="129.54" width="0.1524" layer="91"/>
-<junction x="149.86" y="129.54"/>
 <pinref part="IC1" gate="G$1" pin="RESET"/>
 <wire x1="152.4" y1="152.4" x2="134.62" y2="152.4" width="0.1524" layer="91"/>
@@
 <wire x1="152.4" y1="134.62" x2="134.62" y2="134.62" width="0.1524" layer="91"/>
 <junction x="134.62" y="134.62"/>
+<pinref part="IC1" gate="G$1" pin="AVCC"/>
+<wire x1="152.4" y1="132.08" x2="134.62" y2="132.08" width="0.1524" layer="91"/>
+<junction x="134.62" y="132.08"/>
 </segment>
 </net>
@@
 </sheet>
 </sheets>
+<errors>
+</errors>
 </schematic>
 </drawing>
